File: E3-LED_v2/E3-LED_v2.brd (EAGLE design)
At the start: 10.2 x 19.1 mm, 4 parts

Commit message: Updated BOM and schematic of v2 board with final LED and resistor choice.
Parts:
- R1: value ??? -> DNP
- R2: value ??? -> 180 ohms
Changed lines of the file:
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@@
 </autorouter>
 <elements>
-<element name="R1" library="eagle-ltspice" package="0204/7" value="???" x="5.08" y="8.89">
+<element name="R1" library="eagle-ltspice" package="0204/7" value="DNP" x="5.08" y="8.89">
 <attribute name="SPICEPREFIX" value="R" x="5.08" y="8.89" size="1.778" layer="27" display="off"/>
 <attribute name="SPICEMODEL" value="NONE" x="5.08" y="8.89" size="1.778" layer="27" display="off"/>
@@
 <element name="D1" library="SparkFun-LED" package="LED5MM" value="" x="5.08" y="3.81" rot="R180"/>
 <element name="J1" library="SparkFun-Connectors" package="1X02" value="" x="3.81" y="11.43" rot="MR180"/>
-<element name="R2" library="eagle-ltspice" package="R0603" value="???" x="5.08" y="8.89">
+<element name="R2" library="eagle-ltspice" package="R0603" value="180 ohms" x="5.08" y="8.89">
 <attribute name="SPICEPREFIX" value="R" x="5.08" y="8.89" size="1.778" layer="27" display="off"/>
 <attribute name="SPICEMODEL" value="NONE" x="5.08" y="8.89" size="1.778" layer="27" display="off"/>

Commit message: Tweaked silk.
Parts:
- removed R1: DNP, eagle-ltspice:0204/7
Connections:
- net GND: no longer R1.1
- net N$3: no longer R1.2
Routing:
- net N$3: track 11.6 -> 5.96 mm
- net GND: track 0.00 -> 2.71 mm
Changed lines of the file:
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@@
 LED</text>
 <text x="5.842" y="1.016" size="1.27" layer="22" font="vector" ratio="12" rot="MR0">v2</text>
-<text x="0.889" y="10.16" size="1.016" layer="22" font="vector" ratio="12" rot="MR90">GND</text>
-<text x="8.128" y="10.033" size="1.016" layer="22" font="vector" ratio="12" rot="MR90">+5V</text>
+<text x="0.889" y="3.81" size="1.016" layer="22" font="vector" ratio="12" rot="MR90">GND</text>
+<text x="8.128" y="3.683" size="1.016" layer="22" font="vector" ratio="12" rot="MR90">+5V</text>
 </plain>
 <attributes>
@@
 </autorouter>
 <elements>
-<element name="R1" library="eagle-ltspice" package="0204/7" value="DNP" x="5.08" y="8.89">
-<attribute name="SPICEPREFIX" value="R" x="5.08" y="8.89" size="1.778" layer="27" display="off"/>
-<attribute name="SPICEMODEL" value="NONE" x="5.08" y="8.89" size="1.778" layer="27" display="off"/>
-</element>
 <element name="D1" library="SparkFun-LED" package="LED5MM" value="" x="5.08" y="3.81" rot="R180"/>
 <element name="J1" library="SparkFun-Connectors" package="1X02" value="" x="3.81" y="11.43" rot="MR180"/>
@@
 </polygon>
 <contactref element="J1" pad="1"/>
-<contactref element="R1" pad="1"/>
 <contactref element="R2" pad="1"/>
+<wire x1="4.23" y1="8.89" x2="4.23" y2="11.01" width="0.254" layer="1"/>
+<wire x1="4.23" y1="11.01" x2="3.81" y2="11.43" width="0.254" layer="1"/>
 </signal>
 <signal name="+5V">
@@
 </signal>
 <signal name="N$3">
-<contactref element="R1" pad="2"/>
 <contactref element="D1" pad="K"/>
-<wire x1="3.81" y1="3.81" x2="3.81" y2="6.35" width="0.254" layer="1"/>
-<wire x1="3.81" y1="6.35" x2="5.08" y2="7.62" width="0.254" layer="1"/>
-<wire x1="5.08" y1="7.62" x2="7.62" y2="7.62" width="0.254" layer="1"/>
-<wire x1="7.62" y1="7.62" x2="8.89" y2="8.89" width="0.254" layer="1"/>
+<wire x1="3.81" y1="3.81" x2="3.81" y2="5.08" width="0.254" layer="1"/>
+<wire x1="3.81" y1="5.08" x2="5.93" y2="7.2" width="0.254" layer="1"/>
 <contactref element="R2" pad="2"/>
-<wire x1="5.93" y1="8.89" x2="8.89" y2="8.89" width="0.254" layer="1"/>
+<wire x1="5.93" y1="8.89" x2="5.93" y2="7.2" width="0.254" layer="1"/>
 </signal>
 </signals>
